File: PCB Files/HGC PCB.kicad_pcb (KiCad board)
At the start: 2 copper layers, 174.5 x 69.8 mm, 97 parts, among them J1 MPU6050, J10 Conn_01x07_Pin, J11 Conn_01x07_Pin, J12 Conn_01x04_Pin, J13 Conn_01x07_Pin, J14 USB_C_Receptacle_USB2.0_16P, J15 Conn_01x08_Pin, J16 Conn_01x08_Pin, J17 B2B-XH-A__LF__SN_, J18 B2B-XH-A__LF__SN_, J2 DISPLAY, J3 SDCARD, J4 Conn_01x07_Pin, J5 Conn_01x07_Pin, J6 Conn_01x07_Pin, J7 Conn_01x05_Pin, J8 Conn_01x05_Pin, J9 Conn_01x07_Pin, SW1 SW_SPDT, SW2 SW_Push, SW3 SW_Push, SW4 SW_Push, SW5 SW_Push, SW6 SW_Push, SW7 SW_Push, SW8 SW_Push, U1 STM32F407VGTx, U2 JOYSTICK, U3 AMS1117-3.3, U4 CP2102N-Axx-xQFN28, U5 MP1584EN-LF, Y1 Crystal_GND24

Commit message: Add files via upload
Parts:
- removed the G*** at (211.1, 126.5)
- added G***: LOGO, logos:sra_logo_small_neg, F.Cu at (202.7, 125.8)
- added G***: LOGO, logos:sra_skull_big, B.Cu at (154.5, 102.5)
- added G***: LOGO, Logos:sra_logo_big, B.Cu at (166.2, 109.4)
- added H10: MountingHole, MountingHole:MountingHole_3.2mm_M3, F.Cu at (107.7, 73.5)
- added H4: MountingHole, MountingHole:MountingHole_3.2mm_M3, F.Cu at (84.8, 130.0)
- added H5: MountingHole, MountingHole:MountingHole_3.2mm_M3, F.Cu at (210.8, 130.0)
- added H9: MountingHole, MountingHole:MountingHole_3.2mm_M3, F.Cu at (183.8, 73.5)
- added REF**: WEEE-Logo_8.4x12mm_SilkScreen, Symbol:WEEE-Logo_8.4x12mm_SilkScreen, B.Cu at (213.8, 121.8)
- added REF**: OSHW-Logo_7.5x8mm_SilkScreen, Symbol:OSHW-Logo_7.5x8mm_SilkScreen, B.Cu at (222.0, 119.6)
- added REF**: KiCad-Logo2_6mm_SilkScreen, symbols1:KiCad-Logo2_6mm_SilkScreen, B.Cu at (140.8, 109.5)
- added kibuzzard-668FE423: G***, kibuzzard-668FE423, F.Cu at (149.4, 72.3)
- added kibuzzard-675FDA6A: G***, kibuzzard-675FDA6A, F.Cu at (150.2, 122.0)
- added kibuzzard-68C922B8: G***, kibuzzard-68C922B8, F.Cu at (183.5, 64.7)
- added kibuzzard-68C922D4: G***, kibuzzard-68C922D4, F.Cu at (164.3, 64.8)
- added kibuzzard-68C92324: G***, kibuzzard-68C92324, F.Cu at (120.8, 64.8)
- added kibuzzard-68C923AF: G***, kibuzzard-68C923AF, F.Cu at (135.1, 127.0)
- added kibuzzard-68C923C7: G***, kibuzzard-68C923C7, F.Cu at (168.2, 127.1)
- added kibuzzard-68C923F6: G***, kibuzzard-68C923F6, F.Cu at (197.1, 70.3)
- added kibuzzard-68C92937: G***, kibuzzard-68C92937, F.Cu at (114.9, 127.1)
- added kibuzzard-68C92F98: G***, kibuzzard-68C92F98, F.Cu at (198.7, 92.3)
- added kibuzzard-68C92FA3: G***, kibuzzard-68C92FA3, F.Cu at (198.8, 94.9)
- added kibuzzard-68C92FAB: G***, kibuzzard-68C92FAB, F.Cu at (198.7, 97.4)
- added kibuzzard-68C92FB6: G***, kibuzzard-68C92FB6, F.Cu at (198.5, 99.9)
- added kibuzzard-68C92FBD: G***, kibuzzard-68C92FBD, F.Cu at (198.6, 105.3)
- added kibuzzard-68C92FC5: G***, kibuzzard-68C92FC5, F.Cu at (198.6, 107.8)
- added kibuzzard-68C92FCD: G***, kibuzzard-68C92FCD, F.Cu at (198.6, 110.5)
- added kibuzzard-68C92FD9: G***, kibuzzard-68C92FD9, F.Cu at (198.8, 113.0)
- added kibuzzard-68C92FE3: G***, kibuzzard-68C92FE3, F.Cu at (198.8, 115.5)
- added kibuzzard-68C92FEC: G***, kibuzzard-68C92FEC, F.Cu at (198.8, 118.0)
- added kibuzzard-68C92FF6: G***, kibuzzard-68C92FF6, F.Cu at (198.8, 120.8)
- added kibuzzard-68C93061: G***, kibuzzard-68C93061, F.Cu at (96.8, 69.7)
- added kibuzzard-68C93086: G***, kibuzzard-68C93086, F.Cu at (97.2, 74.7)
- added kibuzzard-68C93097: G***, kibuzzard-68C93097, F.Cu at (97.1, 72.1)
- added kibuzzard-68C930B6: G***, kibuzzard-68C930B6, F.Cu at (97.1, 79.8)
- added kibuzzard-68C930DF: G***, kibuzzard-68C930DF, F.Cu at (96.9, 86.0)
- added kibuzzard-68C930EB: G***, kibuzzard-68C930EB, F.Cu at (97.1, 77.3)
- added kibuzzard-68C93100: G***, kibuzzard-68C93100, F.Cu at (96.8, 88.5)
- added kibuzzard-68C9310A: G***, kibuzzard-68C9310A, F.Cu at (96.9, 91.1)
- added kibuzzard-68C93116: G***, kibuzzard-68C93116, F.Cu at (96.8, 93.6)
- added kibuzzard-68C93123: G***, kibuzzard-68C93123, F.Cu at (96.9, 96.2)
- added kibuzzard-68C9319C: G***, kibuzzard-68C9319C, F.Cu at (214.8, 95.9)
- added kibuzzard-68C931DF: G***, kibuzzard-68C931DF, F.Cu at (224.0, 106.0)
- added kibuzzard-68C931ED: G***, kibuzzard-68C931ED, F.Cu at (205.6, 106.0)
- added kibuzzard-68C9320A: G***, kibuzzard-68C9320A, F.Cu at (215.0, 125.3)
- added kibuzzard-68C93223: G***, kibuzzard-68C93223, F.Cu at (202.0, 82.3)
- added kibuzzard-68C9322C: G***, kibuzzard-68C9322C, F.Cu at (215.7, 82.2)
- added kibuzzard-68C9330F: G***, kibuzzard-68C9330F, F.Cu at (83.2, 89.8)
- added kibuzzard-68C93326: G***, kibuzzard-68C93326, F.Cu at (140.2, 84.1)
- added kibuzzard-68C9333E: G***, kibuzzard-68C9333E, F.Cu at (191.9, 96.1)
- added kibuzzard-68C93356: G***, kibuzzard-68C93356, F.Cu at (103.6, 94.9)
- added kibuzzard-68C938FF: G***, kibuzzard-68C938FF, B.Cu at (122.2, 78.0)
- added kibuzzard-68C939EA: G***, kibuzzard-68C939EA, F.Cu at (106.0, 70.5)
- added kibuzzard-68C93B18: G***, kibuzzard-68C93B18, B.Cu at (129.2, 106.3)
- added kibuzzard-68C93B2B: G***, kibuzzard-68C93B2B, B.Cu at (116.3, 106.3)
- added kibuzzard-68C93D93: G***, kibuzzard-68C93D93, F.Cu at (151.7, 124.6)
- D3: moved to B.Cu
- SW3, SW4, SW5, SW6, SW7, SW8: footprint Button_Switch_SMD:SW_Push_SPST_NO_Alps_SKRK -> Button_Switch_SMD:SW_Push_1P1T_NO_CK_KSC7xxJ
- moved D5 112.1 mm to (210.2, 78.8), turned to 180 degrees
- moved C22 109.7 mm to (213.6, 83.7), turned to 180 degrees
- moved R7 106.4 mm to (209.1, 83.7), turned to 0 degrees
- moved L1 102.9 mm to (216.0, 91.6), turned to -90 degrees
- moved U5 98.8 mm to (210.5, 91.0), turned to 90 degrees
- moved C29 98.0 mm to (216.0, 96.0), turned to -90 degrees
- moved C26 92.9 mm to (211.5, 97.0), turned to 0 degrees
- moved C27 90.1 mm to (207.7, 96.5), turned to 180 degrees
- moved R12 89.9 mm to (211.4, 99.7), turned to 180 degrees
- moved R11 88.9 mm to (203.6, 94.8), turned to -90 degrees
- moved R9 88.1 mm to (212.7, 102.5), turned to 180 degrees
- moved R14 87.1 mm to (199.8, 94.1), turned to -90 degrees
- moved R10 83.2 mm to (207.5, 102.5), turned to 180 degrees
- moved G*** 82.4 mm to (165.6, 88.1)
- moved J17 72.4 mm to (106.1, 66.8)
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Connections:
- SW3 pad 2: /Push1 -> /Push5
- SW4 pad 2: /Push2 -> /Push6
- SW7 pad 2: /Push5 -> /Push1
- SW8 pad 2: /Push6 -> /Push2
Routing:
- net /3.3V: track 37.2 -> 630.0 mm, vias 0 -> 11
- net GND: track 45.6 -> 179.1 mm, vias 0 -> 14
- net /SPI1_SLK: track 8.80 -> 123.7 mm, vias 1 -> 4
- net /V: track 0.00 -> 90.2 mm, vias 0 -> 1
- net /SW: track 0.00 -> 81.6 mm, vias 0 -> 1
- net /H: track 0.00 -> 81.0 mm, vias 0 -> 1
- net /Push5: track 0.00 -> 77.6 mm, vias 0 -> 2
- net /Push3: track 0.00 -> 76.5 mm, vias 0 -> 2
- net /Push1: track 0.00 -> 69.7 mm, vias 0 -> 2
- net /VBUS: track 3.26 -> 72.0 mm, vias 0 -> 4
- net /SPI1_MOSI: track 64.7 -> 130.2 mm, vias 1 -> 3
- net /Push2: track 0.00 -> 63.4 mm, vias 0 -> 2
- net /SPI1_MISO: track 63.9 -> 127.2 mm, vias 1 -> 4
- net /Push4: track 0.00 -> 62.9 mm, vias 0 -> 2
- net /PE2: track 0.00 -> 60.5 mm
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- added copper zone on F.Cu, net /5V
- added copper zone on B.Cu, net GND
- added copper zone on F.Cu, net GND
- removed copper zone on B.Cu, net (none)
Other:
- board size 174.5 x 69.8 mm -> 174.5 x 69.9 mm
- board text added: "BY, MUSTAFA T R ASHISH NERLEKAR PAARTH SHIRSAT AND MENTORS, VISHAL MUTHA PIYUSH PATLE SHAURYA RANE"
- board text added: "Designed by, Ashish N SRA VJTI Mumbai"
- board text added: "R8"
- board text removed: "By, Ashish Nerlekar Paarth Shirsat Mustafa T R"
- board text removed: "DFPLAYER-MINI"
- board text removed: "MPU6050"

Commit message: pcb updated
Parts:
- removed the REF** at (213.8, 121.8)
- removed the REF** at (222.0, 119.6)
- removed the REF** at (140.8, 109.5)
- removed kibuzzard-68C922B8: G***, kibuzzard-68C922B8
- removed kibuzzard-68C92937: G***, kibuzzard-68C92937
- added REF**: WEEE-Logo_5.6x8mm_SilkScreen, Symbol:WEEE-Logo_5.6x8mm_SilkScreen, B.Cu at (218.0, 120.4)
- added REF**: KiCad-Logo2_6mm_SilkScreen, Symbol:KiCad-Logo2_6mm_SilkScreen, B.Cu at (167.0, 110.3)
- added REF**: OSHW-Logo_5.7x6mm_SilkScreen, Symbol:OSHW-Logo_5.7x6mm_SilkScreen, B.Cu at (224.2, 119.1)
- added kibuzzard-68CBCDEB: G***, kibuzzard-68CBCDEB, F.Cu at (114.9, 127.1)
- added kibuzzard-68CBF0D1: G***, kibuzzard-68CBF0D1, F.Cu at (183.9, 64.7)
- C26: value 220pF -> 150pF
- L1: value 10uH -> 15uH
- R12: value 68.1k -> 100k
- R14: value 124k -> 210k
- R7: value 200k -> 100k
- moved G*** 50.2 mm to (207.0, 75.8)
- moved G*** 26.7 mm to (139.6, 111.3)
- moved G*** 10.4 mm to (174.5, 82.7)
- moved G*** 8.37 mm to (174.8, 93.6)
- moved C14 1.94 mm to (139.7, 112.4)
- moved G*** 1.85 mm to (153.3, 101.1)
- moved kibuzzard-668FE423 1.57 mm to (149.3, 73.9)
- moved R2 0.40 mm to (141.1, 96.9)
- moved J14 0.37 mm to (149.5, 67.0)
- moved kibuzzard-68C92324 0.15 mm to (120.7, 64.9)
- moved kibuzzard-68C922D4 0.12 mm to (164.3, 64.6)
- turned SW8 to 0 degrees
Connections:
- C29 pad 1: /3.3V -> /5V
- J15 pad 1: /3.3V -> /5V
- J6 pad 1: /3.3V -> /5V
- J9 pad 1: /PC0 -> /PD4
- J9 pad 2: /PC1 -> /PD3
- L1 pad 2: /3.3V -> /5V
- R14 pad 2: /3.3V -> /5V
- U1 pad 15: /PC0 -> /V
- U1 pad 16: /PC1 -> /H
- U1 pad 84: /V -> /PD3
- U1 pad 85: /H -> /PD4
Routing:
- net /5V: track 10.8 -> 225.1 mm, vias 1 -> 6
- net /PD4: track 0.00 -> 60.3 mm, vias 0 -> 1
- net /PD3: track 0.00 -> 58.4 mm, vias 0 -> 1
- net /PC0: track 53.1 -> 0.00 mm, vias 1 -> 0
- net /PC1: track 49.2 -> 0.00 mm, vias 1 -> 0
- net GND: track 179.1 -> 162.5 mm, vias 14 -> 15
- net /3.3V: track 630.0 -> 620.1 mm, vias 11 -> 8
- net /D+: track 46.7 -> 54.0 mm
- net /V: track 90.2 -> 95.9 mm
- net /Push2: track 63.4 -> 59.4 mm
- net /Push3: track 76.5 -> 80.0 mm, vias 2 -> 3
- net /H: track 81.0 -> 77.8 mm
- net /DC: track 45.5 -> 42.7 mm
- net /sw_boot0: track 35.2 -> 32.4 mm
- net /PB4: track 46.8 -> 49.0 mm
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
Commit message: pcb updated again
Parts:
- removed the G*** at (174.5, 82.7)
- removed the G*** at (174.8, 93.6)
- removed the G*** at (153.3, 101.1)
- removed the G*** at (139.6, 111.3)
- added G***: LOGO, logos:sra_skull_big, F.Cu at (170.6, 90.0)
- added G***: LOGO, Logos:sra_logo_big, F.Cu at (170.4, 79.2)
- added G***: LOGO, Logos:sra_logo_big, B.Cu at (135.4, 107.8)
- added G***: LOGO, logos:sra_skull_big, B.Cu at (149.1, 97.6)
- moved C10 5.45 mm to (159.3, 93.1)
- moved C11 5.45 mm to (155.6, 114.0)
- moved C12 5.45 mm to (135.2, 102.6)
- moved C16 5.45 mm to (133.5, 115.8)
- moved C23 5.45 mm to (174.5, 71.9)
- moved C25 5.45 mm to (164.7, 79.0)
- moved C29 5.45 mm to (211.9, 92.5)
- moved C4 5.45 mm to (141.0, 113.4)
- moved C6 5.45 mm to (159.3, 97.3)
- moved C7 5.45 mm to (135.2, 105.2)
- moved C9 5.45 mm to (139.8, 92.6)
- moved D1 5.45 mm to (178.5, 121.3)
- moved D3 5.45 mm to (144.9, 74.3)
- moved D4 5.45 mm to (172.4, 70.4)
- moved G*** 5.45 mm to (202.9, 72.2)
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Routing:
- net /PE1: track 53.1 -> 55.5 mm
- net /PE3: track 55.7 -> 57.8 mm
- net /PB5: track 49.0 -> 47.3 mm
- net GND: track 162.5 -> 161.2 mm, vias 15 -> 17
- net /5V: track 225.1 -> 226.4 mm
- net /3.3V: track 620.1 -> 621.1 mm
- net /PB8: track 45.9 -> 46.5 mm
- net /PE2: track 61.6 -> 61.0 mm

Commit message: pcb updated for final review
Routing:
- net GND: track 161.2 -> 165.9 mm, vias 17 -> 22
Changed lines of the file:
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@@
+	)
+	(segment
+		(start 131.1 94.41)
+		(end 131.11 94.4)
+		(width 0.5)
+		(layer "F.Cu")
+		(net 1)
 	)
 	(segment
@@
 		(end 141.94 93.75)
 		(width 0.3)
+		(layer "F.Cu")
+		(net 1)
+	)
+	(segment
+		(start 126.43 94.41)
+		(end 131.1 94.41)
+		(width 0.5)
 		(layer "F.Cu")
 		(net 1)
@@
 	)
 	(via
+		(at 115.74 94.61)
+		(size 0.6)
+		(drill 0.3)
+		(layers "F.Cu" "B.Cu")
+		(free yes)
+		(net 1)
+	)
+	(via
 		(at 81.52 79.71)
 		(size 0.6)
@@
 		(drill 0.3)
 		(layers "F.Cu" "B.Cu")
+		(net 1)
+	)
+	(via
+		(at 120.86 107.73)
+		(size 0.6)
+		(drill 0.3)
+		(layers "F.Cu" "B.Cu")
+		(free yes)
+		(net 1)
+	)
+	(via
+		(at 121.22 99.02)
+		(size 0.6)
+		(drill 0.3)
+		(layers "F.Cu" "B.Cu")
+		(free yes)
 		(net 1)
 	)
@@
 		(size 0.6)
 		(drill 0.3)
+		(layers "F.Cu" "B.Cu")
+		(free yes)
+		(net 1)
+	)
+	(via
+		(at 126.43 94.41)
+		(size 0.8)
+		(drill 0.4)
+		(layers "F.Cu" "B.Cu")
+		(free yes)
+		(net 1)
+	)
+	(via
+		(at 120.81 123.5)
+		(size 0.6)
+		(drill 0.3)

Commit message: Add files via upload
Parts:
- removed the G*** at (170.6, 90.0)
- removed the G*** at (170.4, 79.2)
- removed the G*** at (135.4, 107.8)
- removed the G*** at (149.1, 97.6)
- removed kibuzzard-68C938FF: G***, kibuzzard-68C938FF
- added ?: , , F.Cu at (117.2, 105.0)
- added G***: LOGO, logos:sra_skull_big, F.Cu at (172.9, 94.7)
- added G***: LOGO, Logos:sra_logo_big, F.Cu at (172.7, 83.9)
- added G***: LOGO, logos:sra_skull_big, B.Cu at (151.4, 102.3)
- added G***: LOGO, Logos:sra_logo_big, B.Cu at (137.7, 112.5)
- added kibuzzard-68D3B1B5: G***, kibuzzard-68D3B1B5, B.Cu at (119.7, 83.3)
- moved J16 5.26 mm to (129.8, 87.0)
- moved C10 5.25 mm to (161.6, 97.8)
- moved C16 5.25 mm to (135.8, 120.5)
- moved C25 5.25 mm to (167.0, 83.7)
- moved C29 5.25 mm to (214.2, 97.2)
- moved C4 5.25 mm to (143.3, 118.1)
- moved C6 5.25 mm to (161.6, 102.0)
- moved C7 5.25 mm to (137.5, 109.9)
- moved C9 5.25 mm to (142.1, 97.3)
- moved D1 5.25 mm to (180.8, 126.0)
- moved D3 5.25 mm to (147.2, 79.0)
- moved G*** 5.25 mm to (81.9, 83.3)
- moved H8 5.25 mm to (87.9, 69.2)
- moved J2 5.25 mm to (186.9, 113.2)
- moved J6 5.25 mm to (174.1, 68.1)
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Routing:
- net /3.3V: track 621.1 -> 637.4 mm
- net GND: track 165.9 -> 178.3 mm, vias 22 -> 16
- net /VBUS: track 72.1 -> 75.6 mm
- net /PB8: track 46.5 -> 43.5 mm
- net /sw_boot0: track 32.4 -> 35.1 mm
- net /PB4: track 49.0 -> 46.6 mm
- net /12V: track 55.9 -> 57.7 mm
- net /HSE_OUT: track 29.3 -> 27.7 mm
- net /PB9: track 52.8 -> 54.1 mm
- net /PE2: track 61.0 -> 62.3 mm
- net /5V: track 226.4 -> 225.2 mm
- net /PC2: track 45.2 -> 44.3 mm
- net /PB3: track 46.7 -> 45.8 mm
- net /DC: track 42.7 -> 43.6 mm
- net /Push3: track 80.0 -> 79.2 mm
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
Commit message: Add files via upload
Parts:
- removed ?: , 
- removed the G*** at (205.2, 77.0)
- removed J18: B2B-XH-A__LF__SN_, JST:JST_B2B-XH-A__LF__SN_
- removed the REF** at (222.4, 120.2)
- removed the REF** at (165.2, 111.5)
- removed kibuzzard-68C923F6: G***, kibuzzard-68C923F6
- removed kibuzzard-68C931ED: G***, kibuzzard-68C931ED
- removed kibuzzard-68C939EA: G***, kibuzzard-68C939EA
- removed kibuzzard-68C93B18: G***, kibuzzard-68C93B18
- added D8: 5V, LED_SMD:LED_0805_2012Metric, F.Cu at (124.2, 90.9)
- added R18: 0.3k, Resistor_SMD:R_0805_2012Metric, F.Cu at (125.9, 94.2)
- added REF**: KiCad-Logo2_6mm_SilkScreen, symbols1:KiCad-Logo2_6mm_SilkScreen, B.Cu at (213.2, 111.2)
- added REF**: OSHW-Logo2_7.3x6mm_SilkScreen, Symbol:OSHW-Logo2_7.3x6mm_SilkScreen, B.Cu at (221.4, 120.6)
- added kibuzzard-6946C392: G***, kibuzzard-6946C392, F.Cu at (104.4, 70.4)
- added kibuzzard-6946C401: G***, kibuzzard-6946C401, F.Cu at (84.1, 76.2)
- added kibuzzard-6946C61F: G***, kibuzzard-6946C61F, F.Cu at (137.8, 71.7)
- added kibuzzard-694FD5EF: G***, kibuzzard-694FD5EF, F.Cu at (71.7, 95.9)
- added kibuzzard-694FDB00: G***, kibuzzard-694FDB00, F.Cu at (203.8, 107.2)
- C17, C22, C24, C25, C26, C27, C28, C29, D5, D6, D7, J17, L1, R10, R11, R12, R13, R14, R15, R16, R17, R7, R8, R9, kibuzzard-68C93B2B, kibuzzard-68D3B1B5: moved to F.Cu
- C18: footprint Capacitor_SMD:C_0805_2012Metric -> Capacitor_Tantalum_SMD:CP_EIA-3216-10_Kemet-I_HandSolder
- C23: footprint Capacitor_SMD:C_0805_2012Metric -> Capacitor_Tantalum_SMD:CP_EIA-3216-10_Kemet-I_HandSolder; moved to F.Cu
- C5, C6: value 2.2 µF -> 2.2µF
- G***: moved to B.Cu
- J15: footprint Connector_PinSocket_2.54mm:PinSocket_1x08_P2.54mm_Vertical -> Connector_JST:JST_EH_S8B-EH_1x08_P2.50mm_Horizontal; moved to F.Cu
- J16: value Conn_01x08_Pin -> B2B-XH-A__LF__SN_; footprint Connector_PinSocket_2.54mm:PinSocket_1x08_P2.54mm_Vertical -> JST:JST_B2B-XH-A__LF__SN_; moved to F.Cu
- U3: value AMS1117-3.3 -> AMS1117; moved to F.Cu
- U4: value CP2102N-Axx-xQFN28 -> CP2102N; moved to F.Cu
- U5: value MP1584EN-LF -> MP1584; moved to F.Cu
- moved D2 109.6 mm to (185.4, 125.5)
- moved R4 109.6 mm to (189.8, 125.4)
- moved C29 100.7 mm to (113.6, 103.3)
- moved L1 100.6 mm to (113.6, 95.4)
- moved R9 100.4 mm to (111.2, 91.4), turned to -90 degrees
- moved D5 99.3 mm to (110.5, 97.1), turned to -90 degrees
- moved C22 95.7 mm to (116.1, 87.5), turned to 0 degrees
- moved C17 93.5 mm to (112.4, 76.8)
- moved R10 92.6 mm to (113.8, 91.4), turned to 90 degrees
- moved C26 91.5 mm to (118.2, 100.8), turned to 180 degrees
- moved R12 91.4 mm to (118.2, 103.5), turned to 0 degrees
- moved U5 89.5 mm to (119.2, 94.8)
- moved R7 86.5 mm to (120.8, 87.5), turned to 180 degrees
- moved G*** 84.7 mm to (161.8, 111.6), turned to 180 degrees
- moved C27 83.1 mm to (122.8, 100.8), turned to 0 degrees
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- renumbered SW2 to nrst
Connections:
- J16 pad 1: unconnected-(J16-Busy-Pad1) -> /SPK2
- J16 pad 2: unconnected-(J16-USB--Pad2) -> /SPK1
- J17 pad 1: /SPK2 -> GND
- J17 pad 2: /SPK1 -> /12V
Routing:
- net GND: track 178.3 -> 77.6 mm, vias 16 -> 18
- net /3.3V: track 637.4 -> 542.5 mm, vias 8 -> 3
- net /USART3_TX: track 35.4 -> 100.7 mm
- net /USART3_RX: track 39.6 -> 99.4 mm
- net /D+: track 54.0 -> 18.1 mm, vias 4 -> 1
- net /SPK2: track 40.2 -> 10.5 mm, vias 1 -> 0
- net /SPK1: track 41.3 -> 13.9 mm, vias 1 -> 0
- net /D-: track 42.6 -> 19.3 mm
- net /V: track 95.9 -> 74.1 mm, vias 1 -> 2
- net /VBUS: track 75.6 -> 53.9 mm, vias 4 -> 2
- net Net-(U1-VDDA): track 9.42 -> 29.2 mm
- net Net-(J14-CC2): track 24.5 -> 4.89 mm, vias 2 -> 0
- net /5V: track 225.2 -> 206.8 mm, vias 6 -> 1
- net Net-(J14-CC1): track 20.1 -> 4.45 mm, vias 2 -> 0
- net /NRST: track 47.6 -> 62.1 mm
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- removed copper zone on F.Cu, net /5V
Other:
- board text added: "0.1uF"
- board text added: "3V3"
- board text added: "BY, MUSTAFA T R ASHISH NERLEKAR PAARTH SHIRSAT"
- board text removed: "BY, MUSTAFA T R ASHISH NERLEKAR PAARTH SHIRSAT AND MENTORS, VISHAL MUTHA PIYUSH PATLE SHAURYA RANE"
- board text removed: "R8"
