File: PCB Files/HGC PCB.kicad_sch (KiCad schematic)
At the start: 97 parts, among them J1 MPU6050, J10 Conn_01x07_Pin, J11 Conn_01x07_Pin, J12 Conn_01x04_Pin, J13 Conn_01x07_Pin, J14 USB_C_Receptacle_USB2.0_16P, J15 Conn_01x08_Pin, J16 Conn_01x08_Pin, J17 B2B-XH-A__LF__SN_, J18 B2B-XH-A__LF__SN_, J2 DISPLAY, J3 SDCARD, J4 Conn_01x07_Pin, J5 Conn_01x07_Pin, J6 Conn_01x07_Pin, J7 Conn_01x05_Pin, J8 Conn_01x05_Pin, J9 Conn_01x07_Pin, SW1 SW_SPDT, SW2 SW_Push, SW3 SW_Push, SW4 SW_Push, SW5 SW_Push, SW6 SW_Push, SW7 SW_Push, SW8 SW_Push, U1 STM32F407VGTx, U2 JOYSTICK, U3 AMS1117-3.3, U4 CP2102N-Axx-xQFN28, U5 MP1584EN-LF, Y1 Crystal_GND24

Commit message: pcb updated
Parts:
- C26: value 220pF -> 150pF
- L1: value 10uH -> 15uH
- R12: value 68.1k -> 100k
- R14: value 124k -> 210k
- R7: value 200k -> 100k
Connections:
- net 3.3V: no longer C29.1, J15.1 (VCC), J6.1 (Pin_1), L1.2, R14.2
- net 5V: now also C29.1, J15.1 (VCC), J6.1 (Pin_1), L1.2, R14.2
- net H: now also U1.16 (PC1); no longer U1.85 (PD4)
- net V: now also U1.15 (PC0); no longer U1.84 (PD3)
- net PC0 renamed PD4
- net PD4: now also U1.85 (PD4); no longer U1.15 (PC0)
- net PC1 renamed PD3
- net PD3: now also U1.84 (PD3); no longer U1.16 (PC1)
Changed lines of the file:
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@@
 		)
 	)
-	(label "3.3V"
+	(label "5V"
 		(at 228.6 251.46 180)
 		(effects
@@
 		)
 	)
-	(label "PC0"
+	(label "V"
 		(at 170.18 157.48 0)
 		(effects
@@
 		)
 	)
-	(label "3.3V"
+	(label "5V"
 		(at 134.62 236.22 0)
 		(effects
@@
 		)
 	)
-	(label "V"
+	(label "PD3"
 		(at 114.3 144.78 180)
 		(effects
@@
 		)
 	)
-	(label "H"
+	(label "PD4"
 		(at 114.3 147.32 180)
 		(effects
@@
 		)
 	)
-	(label "PC0"
+	(label "PD4"
 		(at 157.48 259.08 0)
 		(effects
@@
 		)
 	)
-	(label "PC1"
+	(label "PD3"
 		(at 157.48 261.62 0)
 		(effects
@@
 		)
 	)
-	(label "PC1"
+	(label "H"
 		(at 170.18 160.02 0)
 		(effects
@@
 	)
 	(label "5V"
-		(at 290.83 205.74 180)
+		(at 289.2225 205.74 180)
 		(effects
 			(font
@@
 		)
 	)
-	(label "3.3V"
+	(label "5V"
 		(at 391.16 172.72 0)
 		(effects
@@
 			)
 		)
-		(property "Value" "10uH"
+		(property "Value" "15uH"
 			(at 377.19 170.4945 90)
 			(effects
@@
 			)
 		)
-		(property "Value" "124k"
+		(property "Value" "210k"
 			(at 356.3582 190.463 90)
 			(effects
@@
 			)
 		)
-		(property "Value" "200k"
-			(at 287.02 187.96 0)
+		(property "Value" "100k"
+			(at 285.8329 186.7401 0)
 			(effects
 				(font
@@
 			)
 		)
-		(property "Value" "68.1k"
-			(at 351.79 177.6038 90)
+		(property "Value" "100k"
+			(at 351.7973 180.3511 90)
 			(effects
 				(font
@@
 			)
 		)
-		(property "Value" "220pF"
+		(property "Value" "150pF"
 			(at 345.9344 177.1245 90)
 			(effects

Commit message: Add files via upload
Parts:
- removed C18: 10uF, Capacitor_SMD:C_0805_2012Metric, symbol Device:C
- removed C23: 22uF, Capacitor_SMD:C_0805_2012Metric, symbol Device:C
- removed J16: Conn_01x08_Pin, Connector_PinSocket_2.54mm:PinSocket_1x08_P2.54mm_Vertical, symbol Connector:Conn_01x08_Pin
- added C18: 10uF, Capacitor_Tantalum_SMD:CP_EIA-3216-10_Kemet-I_HandSolder, symbol Device:C_Polarized
- added C23: 22uF, Capacitor_Tantalum_SMD:CP_EIA-3216-10_Kemet-I_HandSolder, symbol Device:C_Polarized
- added D8: LED, LED_SMD:LED_0805_2012Metric, symbol Device:LED
- added R18: 0.3k, Resistor_SMD:R_0805_2012Metric, symbol Device:R
- J15: footprint Connector_PinSocket_2.54mm:PinSocket_1x08_P2.54mm_Vertical -> Connector_JST:JST_EH_S8B-EH_1x08_P2.50mm_Horizontal
- renumbered H9 to H10, H10 to H4, H4 to H5, H5 to H6, H6 to H7, H7 to H8, H8 to H9, J17 to J16, J18 to J17
Connections:
- net 3.3V: now also C23.1
- net 5V: now also C18.1, R18.2
- net GND: now also C18.2, C23.2, D8.1 (K)
- new net: D8.2 (A), R18.1
- no-connect marks 39 -> 31
